File: Project/TARC Altimeter.kicad_pcb (KiCad board)
At the start: 2 copper layers, 67.1 x 14.2 mm, 20 parts, among them J1 Power Switch, J2 Programmer Breakout (Conn_01x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, Q1 Q_NMOS_GSD, U1 A23_Socket-TARC_Altimeter, U2 ATtiny85-20SU, U3 AP2210-3.3-TARC_Altimeter, U4 BMP280

Commit message: changed VGS pin
Connections:
- U2 pad 2: VGS -> Net-(U2-Pad2)
- U2 pad 3: Net-(U2-Pad3) -> VGS
Routing:
- net Net-(U2-Pad3): track 8.29 -> 0.00 mm
- net VGS: track 29.2 -> 30.6 mm
